File: hardware/button/button.kicad_sch (KiCad schematic)
At the start: 42 parts, among them J1 MODULE_JST_XH_4P, J2 KEYTOP_DISPLAY_I2C, Q1 2SC1815, Q2 2SC1815, Q3 2SC1815, Q4 2SC1815, Q5 2SC1815, Q6 2SC1815, Q7 2SC1815, Q8 2SC1815, SW1 SW_Push, SW2 SW_Push, SW3 SW_Push, SW4 SW_Push, U1 Pico

Commit message: ボタン基板: NeoPixel6個・MXソケット・Pico浮かせ実装・配置と配線
回路図: 側面ストリップをWS2812B 6個(GP9→330Ω)に変更、押下検出はKailh MXソケット1個、PicoはOSC_Shared:Pico_TH40。
PCB: ユーザーがKiCadで配置・配線した保存版。DRCエラー0、パリティは説明フィールドのみ。

Co-Authored-By: Claude Sonnet 5.5 <noreply@anthropic.com>
Parts:
- removed J2: KEYTOP_DISPLAY_I2C, Connector_PinHeader_2.54mm:PinHeader_1x04_P2.54mm_Vertical, symbol Connector_Generic:Conn_01x04
- removed LED1, LED5: OS4WMLA131A (White), LED_THT:LED_D10.0mm, symbol Device:LED
- removed LED2, LED6: OSB56AA131A (Blue), LED_THT:LED_D10.0mm, symbol Device:LED
- removed LED3, LED7: OS5RAAA131A (Red), LED_THT:LED_D10.0mm, symbol Device:LED
- removed LED4, LED8: OS5YAAA131A (Yellow), LED_THT:LED_D10.0mm, symbol Device:LED
- removed Q1, Q2, Q3, Q4, Q5, Q6, Q7, Q8: 2SC1815, Package_TO_SOT_THT:TO-92_Inline, symbol Transistor_BJT:2SC1815
- removed R1, R2, R5, R6: 100, Resistor_THT:R_Axial_DIN0207_L6.3mm_D2.5mm_P10.16mm_Horizontal, symbol Device:R
- removed R3, R4, R7, R8: 150, Resistor_THT:R_Axial_DIN0207_L6.3mm_D2.5mm_P10.16mm_Horizontal, symbol Device:R
- removed RB1, RB2, RB3, RB4, RB5, RB6, RB7, RB8: 4.7k, Resistor_THT:R_Axial_DIN0207_L6.3mm_D2.5mm_P10.16mm_Horizontal, symbol Device:R
- removed SW2, SW3, SW4: SW_Push, Button_Switch_THT:SW_PUSH_6mm, symbol Switch:SW_Push
- removed U1: Pico, RPi_Pico:RPi_Pico_SMD_TH, symbol RPi_Pico:Pico
- added J2: KEYTOP_LCD_SPI, Connector_PinHeader_2.54mm:PinHeader_1x08_P2.54mm_Vertical, symbol Connector_Generic:Conn_01x08
- added NP1, NP2, NP3, NP4, NP5, NP6: WS2812B, LED_SMD:LED_WS2812B_PLCC4_5.0x5.0mm_P3.2mm, symbol LED:WS2812B
- added R10: 330, Resistor_THT:R_Axial_DIN0207_L6.3mm_D2.5mm_P7.62mm_Horizontal, symbol Device:R
- added U1: Pico 2 H, OSC_Shared:RPi_Pico_TH_Headers, symbol OSC_Shared:Pico_TH40
- LED9: footprint LED_THT:LED_D5.0mm -> LED_THT:LED_D3.0mm
- R9: footprint Resistor_THT:R_Axial_DIN0207_L6.3mm_D2.5mm_P10.16mm_Horizontal -> Resistor_THT:R_Axial_DIN0207_L6.3mm_D2.5mm_P7.62mm_Horizontal
- SW1: footprint Button_Switch_THT:SW_PUSH_6mm -> Button_Local:Kailh_socket_MX
Connections:
- net +3.3V: now also J2.1 (Pin_1), U1.36 (3V3)
- net +5V: now also NP1.1 (VDD), NP2.1 (VDD), NP3.1 (VDD), NP4.1 (VDD), NP5.1 (VDD), NP6.1 (VDD), U1.39 (VSYS)
- net GND: now also J2.2 (Pin_2), NP1.3 (VSS), NP2.3 (VSS), NP3.3 (VSS), NP4.3 (VSS), NP5.3 (VSS), NP6.3 (VSS), U1.13 (GND), U1.18 (GND), U1.23 (GND), U1.28 (GND), U1.3 (GND), U1.33 (AGND), U1.38 (GND), U1.8 (GND)
- net BTN: now reaches SW1.2
- net BTN: now also U1.6 (GPIO4)
- net at J1.1 (Pin_1): now also U1.1 (GPIO0)
- net at J1.2 (Pin_2): now also U1.2 (GPIO1)
- net STATUS_LED: now reaches R9.1
- net STATUS_LED: now also U1.20 (GPIO15)
- new net: NP1.4 (DIN), R10.2
- new net: NP5.2 (DOUT), NP6.4 (DIN)
- new net: NP4.2 (DOUT), NP5.4 (DIN)
- new net: NP3.2 (DOUT), NP4.4 (DIN)
- new net: NP2.2 (DOUT), NP3.4 (DIN)
- new net: NP1.2 (DOUT), NP2.4 (DIN)
- new net LCD_BL: J2.8 (Pin_8), U1.29 (GPIO22)
- new net LCD_CLK: J2.4 (Pin_4), U1.24 (GPIO18)
- new net LCD_CS: J2.5 (Pin_5), U1.22 (GPIO17)
- new net LCD_DC: J2.6 (Pin_6), U1.26 (GPIO20)
- new net LCD_DIN: J2.3 (Pin_3), U1.25 (GPIO19)
- new net LCD_RST: J2.7 (Pin_7), U1.27 (GPIO21)
- new net NEO_DIN: R10.1, U1.12 (GPIO9)
- no-connect marks 18 -> 20
Other:
- note added: "J1: host link (UART0 + 5V), bulk cap C1"
- note added: "J2: keytop colour LCD (GC9A01, SPI0)"
- note added: "Press detect: one MX hot-swap switch, GP4"
- note added: "Side strip: 6x WS2812B NeoPixel (GP9 -> 330R -> DIN chain)"
- note added: "Status LED"
