File: hardware/four_button/four_button.kicad_sch (KiCad schematic)
At the start: 20 parts, among them J1 MODULE_JST_XH_4P, SW1 Kailh_socket_MX, SW2 Kailh_socket_MX, SW3 Kailh_socket_MX, SW4 Kailh_socket_MX, SW5 Kailh_socket_MX, SW6 Kailh_socket_MX, SW7 Kailh_socket_MX, SW8 Kailh_socket_MX, SW9 Mode select, U1 Pico 2 H

Commit message: four_button: LEDをWS2812BからSK6812に変更(回路図パッチ)
既存のfour_button.kicad_sch(90ffc76時点)を元に、再生成ではなく直接パッチで
WS2812B->SK6812に差し替え。両部品は物理ピン配置(VDD上/DOUT右/VSS下/DIN左)は
同一だがピン番号が異なる(WS2812B: 1=VDD,2=DOUT,3=VSS,4=DIN / SK6812:
1=VSS,2=DIN,3=VDD,4=DOUT)ため、ワイヤ座標はそのままにlib_id/footprint/
ピン番号マッピングのみ更新。ERC 0件、ネットリスト検証済み。

Co-Authored-By: Claude Sonnet 5 <noreply@anthropic.com>
Parts:
- D1: value WS2812B Red -> SK6812 Red; footprint LED_SMD:LED_WS2812B_PLCC4_5.0x5.0mm_P3.2mm -> LED_SMD:LED_SK6812_PLCC4_5.0x5.0mm_P3.2mm; symbol LED:WS2812B -> LED:SK6812
- D2: value WS2812B Blue -> SK6812 Blue; footprint LED_SMD:LED_WS2812B_PLCC4_5.0x5.0mm_P3.2mm -> LED_SMD:LED_SK6812_PLCC4_5.0x5.0mm_P3.2mm; symbol LED:WS2812B -> LED:SK6812
- D3: value WS2812B Green -> SK6812 Green; footprint LED_SMD:LED_WS2812B_PLCC4_5.0x5.0mm_P3.2mm -> LED_SMD:LED_SK6812_PLCC4_5.0x5.0mm_P3.2mm; symbol LED:WS2812B -> LED:SK6812
- D4: value WS2812B Yellow -> SK6812 Yellow; footprint LED_SMD:LED_WS2812B_PLCC4_5.0x5.0mm_P3.2mm -> LED_SMD:LED_SK6812_PLCC4_5.0x5.0mm_P3.2mm; symbol LED:WS2812B -> LED:SK6812
Connections:
- net +5V: now also D1.3 (VDD), D2.3 (VDD), D3.3 (VDD), D4.3 (VDD); no longer D1.1 (VDD), D2.1 (VDD), D3.1 (VDD), D4.1 (VDD)
- net GND: now also D1.1 (VSS), D2.1 (VSS), D3.1 (VSS), D4.1 (VSS); no longer D1.3 (VSS), D2.3 (VSS), D3.3 (VSS), D4.3 (VSS)
- net at D4.2 (DIN): now also D3.4 (DOUT)
- net at D4.4 (DOUT): no longer D3.2 (DOUT)
- net at R10.2: now also D1.2 (DIN); no longer D1.4 (DIN)
- net at D2.2 (DIN): now also D1.4 (DOUT); no longer D3.4 (DIN)
- net at D2.4 (DOUT): now also D3.2 (DIN); no longer D1.2 (DOUT)
Other:
- note added: "NeoPixel chain (SK6812 x4, red/blue/green/yellow), GP6 via R10"
- note removed: "NeoPixel chain (WS2812B x4, red/blue/green/yellow), GP6 via R10"
Changed lines of the file:
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@@
 			)
 		)
-		(property "Description" "Four-button module MCU (Raspberry Pi Pico 2 H on 2.54mm headers, floating ~2.5mm; 40 header pins only, hub decision 2026-09-30). GP2-5=button inputs (shared between grid and diamond sockets, only one set populated at a time). GP6=NeoPixel data (WS2812B x4 daisy-chained via R10, unused in grid/keypad mode). GP7-9=spare/unused (freed up by the 2026-10-01 NeoPixel switch, previously LEDDRV_B/G/Y). GP10=status LED. GP11=mode-select switch."
+		(property "Description" "Four-button module MCU (Raspberry Pi Pico 2 H on 2.54mm headers, floating ~2.5mm; 40 header pins only, hub decision 2026-09-30). GP2-5=button inputs (shared between grid and diamond sockets, only one set populated at a time). GP6=NeoPixel data (SK6812 x4 daisy-chained via R10, unused in grid/keypad mode). GP7-9=spare/unused (freed up by the 2026-10-01 NeoPixel switch, previously LEDDRV_B/G/Y). GP10=status LED. GP11=mode-select switch."
 			(at 152.4 88.9 0)
 			(hide yes)
@@
 	)
 	(symbol
-		(lib_id "LED:WS2812B")
+		(lib_id "LED:SK6812")
 		(at 342.9 177.8 0)
 		(unit 1)
@@
 			)
 		)
-		(property "Value" "WS2812B Red"
+		(property "Value" "SK6812 Red"
 			(at 342.9 182.88 0)
 			(show_name no)
@@
 			)
 		)
-		(property "Footprint" "LED_SMD:LED_WS2812B_PLCC4_5.0x5.0mm_P3.2mm"
+		(property "Footprint" "LED_SMD:LED_SK6812_PLCC4_5.0x5.0mm_P3.2mm"
 			(at 342.9 177.8 0)
 			(hide yes)
@@
 			)
 		)
-		(property "Description" "Addressable RGB LED (NeoPixel-compatible), Red key. Replaces the discrete LED+2SC1815+resistor driver (2026-10-01, user decision: WS2812B 5050 SMD chosen over SK6812MINI-E -- the latter is already used in complicated_wires but judged too hard to hand-solder; commonising on WS2812B going forward). Daisy-chained GP6->R10->D1->D2->D3->D4 (chain order = dict order Red/Blue/Green/Yellow); firmware addresses each LED by chain position, colour is software-assigned (not fixed by the LED itself). Pin1=VDD(+5V), pin2=DOUT, pin3=VSS(GND), pin4=DIN. Placed near the Red(left) key (not aligned to the switch's LED window -- user decision: thin keycap + indirect lighting, see four_button_design_notes.md)."
+		(property "Description" "Addressable RGB LED (NeoPixel-compatible), Red key. Replaces the discrete LED+2SC1815+resistor driver. 2026-10-01: initially chose WS2812B 5050 SMD over SK6812MINI-E (the latter used in complicated_wires but hard to hand-solder); later changed to the full-size SK6812 5050 (same PLCC4 5.0x5.0mm package/footprint as WS2812B, same physical pin layout, but KiCad's stock SK6812 symbol numbers the pins differently -- pin1=VSS,2=DIN,3=VDD,4=DOUT vs WS2812B's 1=VDD,2=DOUT,3=VSS,4=DIN; verified against both stock library symbols before patching). Daisy-chained GP6->R10->D1->D2->D3->D4 (chain order = dict order Red/Blue/Green/Yellow); firmware addresses each LED by chain position, colour is software-assigned (not fixed by the LED itself). Pin1=VSS(GND), pin2=DIN, pin3=VDD(+5V), pin4=DOUT. Placed near the Red(left) key (not aligned to the switch's LED window -- user decision: thin keycap + indirect lighting, see four_button_design_notes.md)."
 			(at 342.9 177.8 0)
 			(hide yes)
@@
 	)
 	(symbol
-		(lib_id "LED:WS2812B")
+		(lib_id "LED:SK6812")
 		(at 363.22 177.8 0)
 		(unit 1)
@@
 			)
 		)
-		(property "Value" "WS2812B Blue"
+		(property "Value" "SK6812 Blue"
 			(at 363.22 182.88 0)
 			(show_name no)
@@
 			)
 		)
-		(property "Footprint" "LED_SMD:LED_WS2812B_PLCC4_5.0x5.0mm_P3.2mm"
+		(property "Footprint" "LED_SMD:LED_SK6812_PLCC4_5.0x5.0mm_P3.2mm"
 			(at 363.22 177.8 0)
 			(hide yes)
@@
 			)
 		)
-		(property "Description" "Addressable RGB LED (NeoPixel-compatible), Blue key. Replaces the discrete LED+2SC1815+resistor driver (2026-10-01, user decision: WS2812B 5050 SMD chosen over SK6812MINI-E -- the latter is already used in complicated_wires but judged too hard to hand-solder; commonising on WS2812B going forward). Daisy-chained GP6->R10->D1->D2->D3->D4 (chain order = dict order Red/Blue/Green/Yellow); firmware addresses each LED by chain position, colour is software-assigned (not fixed by the LED itself). Pin1=VDD(+5V), pin2=DOUT, pin3=VSS(GND), pin4=DIN. Placed near the Blue(top) key (not aligned to the switch's LED window -- user decision: thin keycap + indirect lighting, see four_button_design_notes.md)."
+		(property "Description" "Addressable RGB LED (NeoPixel-compatible), Blue key. Replaces the discrete LED+2SC1815+resistor driver. 2026-10-01: initially chose WS2812B 5050 SMD over SK6812MINI-E (the latter used in complicated_wires but hard to hand-solder); later changed to the full-size SK6812 5050 (same PLCC4 5.0x5.0mm package/footprint as WS2812B, same physical pin layout, but KiCad's stock SK6812 symbol numbers the pins differently -- pin1=VSS,2=DIN,3=VDD,4=DOUT vs WS2812B's 1=VDD,2=DOUT,3=VSS,4=DIN; verified against both stock library symbols before patching). Daisy-chained GP6->R10->D1->D2->D3->D4 (chain order = dict order Red/Blue/Green/Yellow); firmware addresses each LED by chain position, colour is software-assigned (not fixed by the LED itself). Pin1=VSS(GND), pin2=DIN, pin3=VDD(+5V), pin4=DOUT. Placed near the Blue(top) key (not aligned to the switch's LED window -- user decision: thin keycap + indirect lighting, see four_button_design_notes.md)."
 			(at 363.22 177.8 0)
 			(hide yes)
@@
 	)
 	(symbol
-		(lib_id "LED:WS2812B")
+		(lib_id "LED:SK6812")
 		(at 383.54 177.8 0)
 		(unit 1)
@@
 			)
 		)
-		(property "Value" "WS2812B Green"
+		(property "Value" "SK6812 Green"
 			(at 383.54 182.88 0)
 			(show_name no)
@@
 			)
 		)
-		(property "Footprint" "LED_SMD:LED_WS2812B_PLCC4_5.0x5.0mm_P3.2mm"
+		(property "Footprint" "LED_SMD:LED_SK6812_PLCC4_5.0x5.0mm_P3.2mm"
 			(at 383.54 177.8 0)
 			(hide yes)
@@
 			)
 		)
-		(property "Description" "Addressable RGB LED (NeoPixel-compatible), Green key. Replaces the discrete LED+2SC1815+resistor driver (2026-10-01, user decision: WS2812B 5050 SMD chosen over SK6812MINI-E -- the latter is already used in complicated_wires but judged too hard to hand-solder; commonising on WS2812B going forward). Daisy-chained GP6->R10->D1->D2->D3->D4 (chain order = dict order Red/Blue/Green/Yellow); firmware addresses each LED by chain position, colour is software-assigned (not fixed by the LED itself). Pin1=VDD(+5V), pin2=DOUT, pin3=VSS(GND), pin4=DIN. Placed near the Green(bottom) key (not aligned to the switch's LED window -- user decision: thin keycap + indirect lighting, see four_button_design_notes.md)."
+		(property "Description" "Addressable RGB LED (NeoPixel-compatible), Green key. Replaces the discrete LED+2SC1815+resistor driver. 2026-10-01: initially chose WS2812B 5050 SMD over SK6812MINI-E (the latter used in complicated_wires but hard to hand-solder); later changed to the full-size SK6812 5050 (same PLCC4 5.0x5.0mm package/footprint as WS2812B, same physical pin layout, but KiCad's stock SK6812 symbol numbers the pins differently -- pin1=VSS,2=DIN,3=VDD,4=DOUT vs WS2812B's 1=VDD,2=DOUT,3=VSS,4=DIN; verified against both stock library symbols before patching). Daisy-chained GP6->R10->D1->D2->D3->D4 (chain order = dict order Red/Blue/Green/Yellow); firmware addresses each LED by chain position, colour is software-assigned (not fixed by the LED itself). Pin1=VSS(GND), pin2=DIN, pin3=VDD(+5V), pin4=DOUT. Placed near the Green(bottom) key (not aligned to the switch's LED window -- user decision: thin keycap + indirect lighting, see four_button_design_notes.md)."
 			(at 383.54 177.8 0)
 			(hide yes)
@@
 	)
 	(symbol
-		(lib_id "LED:WS2812B")
+		(lib_id "LED:SK6812")
 		(at 403.86 177.8 0)
 		(unit 1)
@@
 			)
 		)
-		(property "Value" "WS2812B Yellow"
+		(property "Value" "SK6812 Yellow"
 			(at 403.86 182.88 0)
 			(show_name no)
@@
 			)
 		)
-		(property "Footprint" "LED_SMD:LED_WS2812B_PLCC4_5.0x5.0mm_P3.2mm"
+		(property "Footprint" "LED_SMD:LED_SK6812_PLCC4_5.0x5.0mm_P3.2mm"
 			(at 403.86 177.8 0)
 			(hide yes)
@@
 			)
 		)
-		(property "Description" "Addressable RGB LED (NeoPixel-compatible), Yellow key. Replaces the discrete LED+2SC1815+resistor driver (2026-10-01, user decision: WS2812B 5050 SMD chosen over SK6812MINI-E -- the latter is already used in complicated_wires but judged too hard to hand-solder; commonising on WS2812B going forward). Daisy-chained GP6->R10->D1->D2->D3->D4 (chain order = dict order Red/Blue/Green/Yellow); firmware addresses each LED by chain position, colour is software-assigned (not fixed by the LED itself). Pin1=VDD(+5V), pin2=DOUT, pin3=VSS(GND), pin4=DIN. Placed near the Yellow(right) key (not aligned to the switch's LED window -- user decision: thin keycap + indirect lighting, see four_button_design_notes.md)."
+		(property "Description" "Addressable RGB LED (NeoPixel-compatible), Yellow key. Replaces the discrete LED+2SC1815+resistor driver. 2026-10-01: initially chose WS2812B 5050 SMD over SK6812MINI-E (the latter used in complicated_wires but hard to hand-solder); later changed to the full-size SK6812 5050 (same PLCC4 5.0x5.0mm package/footprint as WS2812B, same physical pin layout, but KiCad's stock SK6812 symbol numbers the pins differently -- pin1=VSS,2=DIN,3=VDD,4=DOUT vs WS2812B's 1=VDD,2=DOUT,3=VSS,4=DIN; verified against both stock library symbols before patching). Daisy-chained GP6->R10->D1->D2->D3->D4 (chain order = dict order Red/Blue/Green/Yellow); firmware addresses each LED by chain position, colour is software-assigned (not fixed by the LED itself). Pin1=VSS(GND), pin2=DIN, pin3=VDD(+5V), pin4=DOUT. Placed near the Yellow(right) key (not aligned to the switch's LED window -- user decision: thin keycap + indirect lighting, see four_button_design_notes.md)."
 			(at 403.86 177.8 0)
 			(hide yes)
@@
 		)
 	)
-	(text "NeoPixel chain (WS2812B x4, red/blue/green/yellow), GP6 via R10"
+	(text "NeoPixel chain (SK6812 x4, red/blue/green/yellow), GP6 via R10"
 		(exclude_from_sim no)
 		(at 312.42 165.1 0)
